File: OrionV2V3_rp2040.kicad_sch (KiCad schematic)
At the start: 290 parts, among them J1 USB_C_Receptacle_USB2.0_16P, J3 USB_C_Receptacle_USB2.0_16P, U1 XC6206PxxxMR, U2 W25Q128JVS, U3 RP2040, U4 SRV05-4, Y1 ABM8-272-T3

Commit message: V1.1
Parts:
- renumbered LC28 to LC1, LC5 to LC10, LC26 to LC11, LC6 to LC12, LC7 to LC13, LC8 to LC14, LC9 to LC15, LC10 to LC16, LC36 to LC17, LC37 to LC18, LC11 to LC19, LC29 to LC2, LC33 to LC20, LC34 to LC21, LC35 to LC22, LC12 to LC23, LC13 to LC24, LC14 to LC25, LC15 to LC26, LC16 to LC28, LC39 to LC29, LC30 to LC3, LC17 to LC30, LC18 to LC31, LC19 to LC32, LC20 to LC33, LC21 to LC34, LC22 to LC35, LC23 to LC36, LC24 to LC37, LC25 to LC38, LC38 to LC39, LC31 to LC4, LC32 to LC5, LC1 to LC6, LC2 to LC7, LC3 to LC8, LC4 to LC9, ULED28 to ULED1, ULED5 to ULED10, ULED26 to ULED11, ULED6 to ULED12, ULED7 to ULED13, ULED8 to ULED14, ULED9 to ULED15, ULED10 to ULED16, ULED36 to ULED17, ULED37 to ULED18, ULED11 to ULED19, ULED29 to ULED2, ULED33 to ULED20, ULED34 to ULED21, ULED35 to ULED22, ULED12 to ULED23, ULED13 to ULED24, ULED14 to ULED25, ULED15 to ULED26, ULED16 to ULED28, ULED39 to ULED29, ULED30 to ULED3, ULED17 to ULED30, ULED18 to ULED31, ULED19 to ULED32, ULED20 to ULED33, ULED21 to ULED34, ULED22 to ULED35, ULED23 to ULED36, ULED24 to ULED37, ULED25 to ULED38, ULED38 to ULED39, ULED31 to ULED4, ULED32 to ULED5, ULED1 to ULED6, ULED2 to ULED7, ULED3 to ULED8, ULED4 to ULED9
Connections:
- net Neopixel: now reaches R11.2, U3.39 (GPIO27_ADC1)
Other:
- moved on the sheet: C13, C14, F1, J1, J3, LC17, LC18, LC19, LC20, LC21, LC22, LC23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

Commit message: V1.3
Parts:
- removed U1: XC6206PxxxMR, Package_TO_SOT_SMD:SOT-23, symbol Regulator_Linear:XC6206PxxxMR
- added C18: 470pF, Capacitor_SMD:C_0603_1608Metric, symbol Device:C_Small
- added U1: MIC5219-3.3YM5, Package_TO_SOT_SMD:SOT-23-5, symbol Regulator_Linear:MIC5219-3.3YM5
- C13: value 1u -> 2.2uF
- C14: value 1u -> 1uF
- ULED1, ULED11, ULED2, ULED20, ULED21, ULED22, ULED27, ULED3, ULED4, ULED5: footprint ScottoKeebs_Components:LED_SK6812MINI-E_clrce -> ScottoKeebs_Components:LED_SK6812MINI
Connections:
- net +3V3: now also C13.1, U1.5 (OUT); no longer C14.1
- net +5V: now also C14.1, U1.1 (IN), U1.3 (EN); no longer C13.1
- net GND: now also C18.2, U1.2 (GND)
- new net: C18.1, U1.4 (BP)

Commit message: V1.4
Connections:
- net DM: now also U4.1 (IO1); no longer U4.4 (IO3)
- net DP: now also U4.6 (IO4); no longer U4.3 (IO2)
- no-connect marks 7 -> 5
Changed lines of the file:
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@@
 	)
 	(no_connect
-		(at 167.64 125.73)
-	)
-	(no_connect
-		(at 167.64 130.81)
-	)
-	(no_connect
 		(at 274.32 198.12)
 	)
@@
 	(global_label "DM"
 		(shape input)
-		(at 193.04 130.81 0)
+		(at 167.64 125.73 180)
 		(fields_autoplaced yes)
 		(effects
@@
 				(size 1.27 1.27)
 			)
-			(justify left)
+			(justify right)
 		)
 		(property "Intersheetrefs" "${INTERSHEET_REFS}"
-			(at 198.7466 130.81 0)
+			(at 161.9334 125.73 0)
 			(effects
 				(font
 					(size 1.27 1.27)
 				)
-				(justify left)
+				(justify right)
 				(hide yes)
 			)
@@
 	(global_label "DP"
 		(shape input)
-		(at 193.04 125.73 0)
+		(at 167.64 130.81 180)
 		(fields_autoplaced yes)
 		(effects
@@
 				(size 1.27 1.27)
 			)
-			(justify left)
+			(justify right)
 		)
 		(property "Intersheetrefs" "${INTERSHEET_REFS}"
-			(at 198.5652 125.73 0)
+			(at 162.1148 130.81 0)
 			(effects
 				(font
 					(size 1.27 1.27)
 				)
-				(justify left)
+				(justify right)
 				(hide yes)
 			)
